Commit message: fixed bugs

File: lunar_excavator_description/urdf/lunar_excavator.urdf (robot description, URDF)
Before this commit: robot excavator, 9 links, 8 joints
Links:
- link body: mass 2000.0 -> 1916.2173; geometry collision mesh filename=package://lunar_excavator_description/meshes/main_body_simp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; visual mesh filename=package://lunar_excavator_description/meshes/main_body.stl
